File: boards/PCB_Separated/core.brd (EAGLE design)
At the start: 5 parts, among them U1 STM32F10XRXT6

Commit message: Modify Board. Core and FTDI become one file
Parts:
- added IC1: FT232RL, ftdichip:SSOP28
- added IN, OUT: (no value), pinhead:1X04
Connections:
- new net DM: IC1.16, IN.3
- new net DP: IC1.15, IN.2
- new net GND: IC1.21
- new net RX: IC1.5, OUT.2
- new net TX: IC1.1, OUT.1
- new net VCC: IC1.20, IN.4
- net VDD: now also IC1.17, IC1.4, OUT.4
- net VSS: now also IC1.18, IC1.25, IC1.26, IC1.7, IN.1, OUT.3
Routing:
- net VSS: track 291.7 -> 340.0 mm
- net VDD: track 184.3 -> 223.3 mm
- net VCC: track 0.00 -> 8.73 mm
- net DM: track 0.00 -> 8.02 mm
- net DP: track 0.00 -> 6.49 mm
- net TX: track 0.00 -> 5.44 mm
- net RX: track 0.00 -> 5.41 mm
- added copper zone on layer 16, net N$2
Changed lines of the file:
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@@
 <element name="JP3" library="pinhead" package="1X16" value="" x="29.21" y="39.37" rot="R90"/>
 <element name="JP4" library="pinhead" package="1X16" value="" x="50.8" y="60.96"/>
+<element name="IC1" library="ftdichip" package="SSOP28" value="FT232RL" x="87.63" y="52.07" rot="MR0">
+<attribute name="OC_NEWARK" value="91K9918" x="87.63" y="52.07" size="1.778" layer="28" rot="MR0" display="off"/>
+<attribute name="MPN" value="FT232RL" x="87.63" y="52.07" size="1.778" layer="28" rot="MR0" display="off"/>
+<attribute name="MF" value="" x="87.63" y="52.07" size="1.778" layer="28" rot="MR0" display="off"/>
+<attribute name="OC_FARNELL" value="1146032" x="87.63" y="52.07" size="1.778" layer="28" rot="MR0" display="off"/>
+</element>
+<element name="IN" library="pinhead" package="1X04" value="" x="87.63" y="60.96"/>
+<element name="OUT" library="pinhead" package="1X04" value="" x="87.63" y="43.18" rot="R180"/>
 </elements>
 <signals>
@@
 <wire x1="41.91" y1="17.78" x2="41.91" y2="15.24" width="0.3048" layer="16"/>
 <wire x1="67.31" y1="17.78" x2="67.31" y2="15.24" width="0.3048" layer="16"/>
+<contactref element="IC1" pad="25"/>
+<contactref element="IC1" pad="26"/>
+<contactref element="IC1" pad="7"/>
+<contactref element="IC1" pad="18"/>
+<contactref element="IN" pad="1"/>
+<contactref element="OUT" pad="3"/>
+<wire x1="87.955" y1="48.445" x2="87.955" y2="47.315" width="0.4064" layer="16"/>
+<wire x1="87.955" y1="47.315" x2="86.36" y2="45.72" width="0.4064" layer="16"/>
+<wire x1="86.36" y1="45.72" x2="86.36" y2="43.18" width="0.4064" layer="16"/>
+<wire x1="85.355" y1="55.695" x2="85.355" y2="53.075" width="0.4064" layer="16"/>
+<wire x1="85.355" y1="53.075" x2="86.36" y2="52.07" width="0.4064" layer="16"/>
+<wire x1="86.36" y1="52.07" x2="87.63" y2="52.07" width="0.4064" layer="16"/>
+<wire x1="87.63" y1="52.07" x2="90.17" y2="52.07" width="0.4064" layer="16"/>
+<wire x1="89.905" y1="55.695" x2="89.905" y2="52.335" width="0.4064" layer="16"/>
+<wire x1="89.905" y1="52.335" x2="90.17" y2="52.07" width="0.4064" layer="16"/>
+<wire x1="90.555" y1="55.695" x2="90.555" y2="52.455" width="0.4064" layer="16"/>
+<wire x1="90.555" y1="52.455" x2="90.17" y2="52.07" width="0.4064" layer="16"/>
+<wire x1="87.955" y1="48.445" x2="87.955" y2="51.745" width="0.4064" layer="16"/>
+<wire x1="87.955" y1="51.745" x2="87.63" y2="52.07" width="0.4064" layer="16"/>
+<wire x1="83.82" y1="60.96" x2="83.82" y2="62.23" width="0.4064" layer="16"/>
+<wire x1="83.82" y1="62.23" x2="85.09" y2="63.5" width="0.4064" layer="16"/>
+<wire x1="85.09" y1="63.5" x2="91.44" y2="63.5" width="0.4064" layer="16"/>
+<wire x1="91.44" y1="63.5" x2="92.71" y2="62.23" width="0.4064" layer="16"/>
+<wire x1="92.71" y1="62.23" x2="92.71" y2="53.34" width="0.4064" layer="16"/>
+<wire x1="92.71" y1="53.34" x2="91.44" y2="52.07" width="0.4064" layer="16"/>
+<wire x1="91.44" y1="52.07" x2="90.17" y2="52.07" width="0.4064" layer="16"/>
+<wire x1="74.93" y1="62.23" x2="83.82" y2="62.23" width="0" layer="19" extent="16-16"/>
 </signal>
 <signal name="VDD">
@@
 <wire x1="56.5" y1="37.12" x2="53.84" y2="37.12" width="0.3048" layer="16"/>
 <wire x1="53.84" y1="37.12" x2="53.55" y2="36.83" width="0.3048" layer="16"/>
+<contactref element="IC1" pad="17"/>
+<contactref element="IC1" pad="4"/>
+<contactref element="OUT" pad="4"/>
+<wire x1="89.905" y1="48.445" x2="89.905" y2="50.535" width="0.4064" layer="16"/>
+<wire x1="89.905" y1="50.535" x2="90.17" y2="50.8" width="0.4064" layer="16"/>
+<wire x1="90.17" y1="50.8" x2="92.71" y2="50.8" width="0.4064" layer="16"/>
+<wire x1="92.71" y1="50.8" x2="92.71" y2="41.91" width="0.4064" layer="16"/>
+<wire x1="92.71" y1="41.91" x2="91.44" y2="40.64" width="0.4064" layer="16"/>
+<wire x1="91.44" y1="40.64" x2="85.09" y2="40.64" width="0.4064" layer="16"/>
+<wire x1="85.09" y1="40.64" x2="83.82" y2="41.91" width="0.4064" layer="16"/>
+<wire x1="83.82" y1="41.91" x2="83.82" y2="43.18" width="0.4064" layer="16"/>
+<wire x1="84.705" y1="55.695" x2="84.705" y2="52.955" width="0.4064" layer="16"/>
+<wire x1="84.705" y1="52.955" x2="82.55" y2="50.8" width="0.4064" layer="16"/>
+<wire x1="82.55" y1="50.8" x2="82.55" y2="44.45" width="0.4064" layer="16"/>
+<wire x1="82.55" y1="44.45" x2="83.82" y2="43.18" width="0.4064" layer="16"/>
+<wire x1="72.39" y1="58.42" x2="84.705" y2="55.695" width="0" layer="19" extent="16-16"/>
 </signal>
 <signal name="P14">
@@
 </polygon>
 </signal>
+<signal name="GND">
+<contactref element="IC1" pad="21"/>
+</signal>
+<signal name="VCC">
+<contactref element="IC1" pad="20"/>
+<contactref element="IN" pad="4"/>
+<wire x1="86.655" y1="55.695" x2="86.655" y2="57.445" width="0.4064" layer="16"/>
+<wire x1="86.655" y1="57.445" x2="87.63" y2="58.42" width="0.4064" layer="16"/>
+<wire x1="87.63" y1="58.42" x2="90.17" y2="58.42" width="0.4064" layer="16"/>
+<wire x1="90.17" y1="58.42" x2="91.44" y2="59.69" width="0.4064" layer="16"/>
+<wire x1="91.44" y1="59.69" x2="91.44" y2="60.96" width="0.4064" layer="16"/>
+</signal>
+<signal name="DP">
+<contactref element="IC1" pad="15"/>
+<contactref element="IN" pad="2"/>
+<wire x1="83.405" y1="55.695" x2="83.405" y2="58.005" width="0.4064" layer="16"/>
+<wire x1="83.405" y1="58.005" x2="86.36" y2="60.96" width="0.4064" layer="16"/>
+</signal>
+<signal name="DM">
+<contactref element="IC1" pad="16"/>
+<contactref element="IN" pad="3"/>
+<wire x1="84.055" y1="55.695" x2="84.055" y2="57.385" width="0.4064" layer="16"/>
+<wire x1="84.055" y1="57.385" x2="85.09" y2="58.42" width="0.4064" layer="16"/>
+<wire x1="85.09" y1="58.42" x2="86.36" y2="58.42" width="0.4064" layer="16"/>
+<wire x1="86.36" y1="58.42" x2="88.9" y2="60.96" width="0.4064" layer="16"/>
+</signal>
+<signal name="TX">
+<contactref element="IC1" pad="1"/>
+<contactref element="OUT" pad="1"/>
+<wire x1="91.855" y1="48.445" x2="91.855" y2="43.595" width="0.4064" layer="16"/>
+<wire x1="91.855" y1="43.595" x2="91.44" y2="43.18" width="0.4064" layer="16"/>
+</signal>
+<signal name="RX">
+<contactref element="IC1" pad="5"/>
+<contactref element="OUT" pad="2"/>
+<wire x1="89.255" y1="48.445" x2="89.255" y2="43.535" width="0.4064" layer="16"/>
+<wire x1="89.255" y1="43.535" x2="88.9" y2="43.18" width="0.4064" layer="16"/>
+</signal>
+<signal name="N$2">
+<polygon width="0.4064" layer="16" isolate="0.6096">
+<vertex x="81.28" y="64.77"/>
+<vertex x="93.98" y="64.77"/>
+<vertex x="93.98" y="39.37"/>
+<vertex x="81.28" y="39.37"/>
+</polygon>
+</signal>

Commit message: -delete a useless sch pics -add ecu io pins diagram -add a GND to VSS line on FTDI. Hopefully internally connected with other GND pins -progress new separated ecu board.
Connections:
- removed net GND: IC1.21
- net VSS: now also IC1.21
Changed lines of the file:
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@@
 <wire x1="92.71" y1="53.34" x2="91.44" y2="52.07" width="0.4064" layer="16"/>
 <wire x1="91.44" y1="52.07" x2="90.17" y2="52.07" width="0.4064" layer="16"/>
+<contactref element="IC1" pad="21"/>
+<wire x1="85.355" y1="55.695" x2="87.305" y2="55.695" width="0" layer="19" extent="16-16"/>
 <wire x1="74.93" y1="62.23" x2="83.82" y2="62.23" width="0" layer="19" extent="16-16"/>
 </signal>
@@
 </polygon>
 </signal>
-<signal name="GND">
-<contactref element="IC1" pad="21"/>
-</signal>
 <signal name="VCC">
