File: boards/PCB_Separated/connector.brd (EAGLE design)
At the start: 3 parts

Commit message: add label on connector design
Connections:
- net N$1 renamed NO_USE-TPS
- net N$2 renamed IGN1-ICU
- net N$3 renamed INJ1-NO_USE
- net N$4 renamed IACB-VSS
- net N$5 renamed IACD-GND
- net N$6 renamed INJ2-NO_USE
- net N$7 renamed IGN2-VSS
- net N$8 renamed IACA-VCC
- net N$9 renamed IACC-V12
Changed lines of the file:
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@@
 </elements>
 <signals>
-<signal name="N$1">
+<signal name="NO_USE-TPS">
 <contactref element="INA" pad="3"/>
 <contactref element="X1" pad="3"/>
@@
 <wire x1="35.687" y1="37.973" x2="35.56" y2="38.1" width="0.6096" layer="16"/>
 </signal>
-<signal name="N$2">
+<signal name="IGN1-ICU">
 <contactref element="INA" pad="4"/>
 <contactref element="X1" pad="4"/>
@@
 <wire x1="35.6108" y1="33.147" x2="35.56" y2="33.0962" width="0.6096" layer="16"/>
 </signal>
-<signal name="N$3">
+<signal name="INJ1-NO_USE">
 <contactref element="INA" pad="5"/>
 <contactref element="X1" pad="5"/>
@@
 <wire x1="35.6616" y1="28.194" x2="35.56" y2="28.0924" width="0.6096" layer="16"/>
 </signal>
-<signal name="N$4">
+<signal name="IACB-VSS">
 <contactref element="INA" pad="2"/>
 <contactref element="X1" pad="2"/>
@@
 <wire x1="35.6362" y1="43.18" x2="35.56" y2="43.1038" width="0.6096" layer="16"/>
 </signal>
-<signal name="N$5">
+<signal name="IACD-GND">
 <contactref element="INA" pad="1"/>
 <contactref element="X1" pad="1"/>
@@
 <wire x1="46.482" y1="48.133" x2="35.56" y2="48.133" width="0.6096" layer="16"/>
 </signal>
-<signal name="N$6">
+<signal name="INJ2-NO_USE">
 <contactref element="X1" pad="9"/>
 <contactref element="INB" pad="1"/>
@@
 <wire x1="43.7134" y1="30.48" x2="43.688" y2="30.4546" width="0.6096" layer="16"/>
 </signal>
-<signal name="N$7">
+<signal name="IGN2-VSS">
 <contactref element="X1" pad="8"/>
 <contactref element="INB" pad="2"/>
@@
 <wire x1="44.8056" y1="36.6014" x2="43.688" y2="35.4838" width="0.6096" layer="16"/>
 </signal>
-<signal name="N$8">
+<signal name="IACA-VCC">
 <contactref element="X1" pad="7"/>
 <contactref element="INB" pad="3"/>
@@
 <wire x1="44.8056" y1="39.3446" x2="43.688" y2="40.4622" width="0.6096" layer="16"/>
 </signal>
-<signal name="N$9">
+<signal name="IACC-V12">
 <contactref element="X1" pad="6"/>
 <contactref element="INB" pad="4"/>
