File: boards/PCB_Separated/iac_driver.brd (EAGLE design)
At the start: 8 parts, among them IC1 L293D

Commit message: IAC progress. Valve already driven, but there a problem with voltage while USB connected to PC
Connections:
- net IACA_IN: now also IC1.2; no longer IC1.3
- net IACA_OUT: now also IC1.3; no longer IC1.2
- net IACD_IN: now also IC1.15; no longer IC1.14
- net IACD_OUT: now also IC1.14; no longer IC1.15
Routing:
- net VCC: track 80.4 -> 94.0 mm
- net IACA_OUT: track 37.3 -> 47.5 mm
- net IACD_OUT: track 38.3 -> 46.8 mm
- net GND: track 35.2 -> 28.9 mm
- net IACD_IN: track 25.6 -> 28.6 mm
- net IACA_IN: track 25.1 -> 27.7 mm
- net V12: track 80.2 -> 82.1 mm
Changed lines of the file:
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@@
 <contactref element="R4" pad="2"/>
 <contactref element="POWER" pad="2"/>
-<wire x1="44.45" y1="52.07" x2="49.657" y2="52.07" width="0.4064" layer="16"/>
 <wire x1="49.657" y1="52.07" x2="52.07" y2="52.07" width="0.4064" layer="16"/>
 <wire x1="55.118" y1="53.34" x2="53.34" y2="53.34" width="0.4064" layer="16"/>
 <wire x1="53.34" y1="53.34" x2="52.07" y2="52.07" width="0.4064" layer="16"/>
 <wire x1="41.529" y1="53.594" x2="42.926" y2="53.594" width="0.4064" layer="16"/>
-<wire x1="42.926" y1="53.594" x2="44.45" y2="52.07" width="0.4064" layer="16"/>
 <wire x1="52.07" y1="34.29" x2="53.721" y2="34.29" width="0.4064" layer="16"/>
 <wire x1="53.721" y1="34.29" x2="55.372" y2="32.639" width="0.4064" layer="16"/>
@@
 <wire x1="54.61" y1="41.656" x2="54.61" y2="44.069" width="0.4064" layer="16"/>
 <wire x1="54.61" y1="44.069" x2="54.737" y2="44.196" width="0.4064" layer="16"/>
+<wire x1="44.45" y1="52.07" x2="42.926" y2="53.594" width="0.4064" layer="16"/>
+<wire x1="41.529" y1="53.594" x2="41.021" y2="53.594" width="0.4064" layer="16"/>
+<wire x1="41.021" y1="53.594" x2="40.386" y2="54.229" width="0.4064" layer="16"/>
+<wire x1="40.386" y1="54.229" x2="40.386" y2="60.579" width="0.4064" layer="16"/>
+<wire x1="40.386" y1="60.579" x2="41.275" y2="61.468" width="0.4064" layer="16"/>
+<wire x1="41.275" y1="61.468" x2="47.879" y2="61.468" width="0.4064" layer="16"/>
+<wire x1="47.879" y1="61.468" x2="48.387" y2="60.96" width="0.4064" layer="16"/>
+<wire x1="48.387" y1="60.96" x2="48.387" y2="58.547" width="0.4064" layer="16"/>
 </signal>
 <signal name="GND">
@@
 <contactref element="IC1" pad="12"/>
 <contactref element="POWER" pad="3"/>
-<wire x1="44.45" y1="44.45" x2="47.498" y2="44.45" width="0.4064" layer="16"/>
-<wire x1="47.498" y1="44.45" x2="52.07" y2="44.45" width="0.4064" layer="16"/>
 <wire x1="44.45" y1="41.91" x2="44.45" y2="44.45" width="0.4064" layer="16"/>
 <wire x1="52.07" y1="41.91" x2="52.07" y2="44.45" width="0.4064" layer="16"/>
-<wire x1="43.3832" y1="58.547" x2="43.3832" y2="58.2422" width="0.4064" layer="16"/>
-<wire x1="43.3832" y1="58.2422" x2="39.878" y2="54.737" width="0.4064" layer="16"/>
-<wire x1="39.878" y1="54.737" x2="39.878" y2="51.562" width="0.4064" layer="16"/>
-<wire x1="39.878" y1="51.562" x2="40.64" y2="50.8" width="0.4064" layer="16"/>
-<wire x1="40.64" y1="50.8" x2="47.117" y2="50.8" width="0.4064" layer="16"/>
-<wire x1="47.117" y1="50.8" x2="47.498" y2="50.419" width="0.4064" layer="16"/>
-<wire x1="47.498" y1="50.419" x2="47.498" y2="44.45" width="0.4064" layer="16"/>
+<wire x1="43.3832" y1="58.547" x2="43.3832" y2="57.5818" width="0.4064" layer="16"/>
+<wire x1="43.3832" y1="57.5818" x2="47.371" y2="53.594" width="0.4064" layer="16"/>
+<wire x1="47.371" y1="53.594" x2="47.371" y2="51.562" width="0.4064" layer="16"/>
+<wire x1="47.371" y1="51.562" x2="47.752" y2="51.181" width="0.4064" layer="16"/>
+<wire x1="47.752" y1="51.181" x2="47.752" y2="45.085" width="0.4064" layer="16"/>
+<wire x1="47.752" y1="45.085" x2="47.117" y2="44.45" width="0.4064" layer="16"/>
+<wire x1="47.117" y1="44.45" x2="44.45" y2="44.45" width="0.4064" layer="16"/>
+<wire x1="52.07" y1="44.45" x2="47.117" y2="44.45" width="0.4064" layer="16"/>
 </signal>
 <signal name="V12">
@@
 <wire x1="53.3908" y1="58.547" x2="53.721" y2="58.547" width="0.4064" layer="16"/>
 <wire x1="53.721" y1="58.547" x2="60.198" y2="52.07" width="0.4064" layer="16"/>
-<wire x1="60.198" y1="20.32" x2="54.737" y2="14.859" width="0.4064" layer="16"/>
-<wire x1="54.737" y1="14.859" x2="43.815" y2="14.859" width="0.4064" layer="16"/>
+<wire x1="58.039" y1="14.859" x2="43.815" y2="14.859" width="0.4064" layer="16"/>
 <wire x1="43.815" y1="14.859" x2="43.053" y2="15.621" width="0.4064" layer="16"/>
 <wire x1="43.053" y1="15.621" x2="43.053" y2="27.94" width="0.4064" layer="16"/>
@@
 <wire x1="44.069" y1="28.956" x2="44.069" y2="33.909" width="0.4064" layer="16"/>
 <wire x1="44.069" y1="33.909" x2="44.45" y2="34.29" width="0.4064" layer="16"/>
-<wire x1="60.198" y1="52.07" x2="60.198" y2="20.32" width="0.4064" layer="16"/>
+<wire x1="60.198" y1="52.07" x2="60.198" y2="17.018" width="0.4064" layer="16"/>
+<wire x1="58.039" y1="14.859" x2="60.198" y2="17.018" width="0.4064" layer="16"/>
 </signal>
 <signal name="IACA_OUT">
-<contactref element="IC1" pad="2"/>
 <contactref element="OUTPUT" pad="1"/>
-<wire x1="44.45" y1="49.53" x2="43.053" y2="49.53" width="0.4064" layer="16"/>
-<wire x1="43.053" y1="49.53" x2="37.084" y2="43.561" width="0.4064" layer="16"/>
-<wire x1="37.084" y1="43.561" x2="37.084" y2="20.9296" width="0.4064" layer="16"/>
+<wire x1="37.084" y1="47.752" x2="37.084" y2="20.9296" width="0.4064" layer="16"/>
 <wire x1="37.084" y1="20.9296" x2="40.4876" y2="17.526" width="0.4064" layer="16"/>
+<contactref element="IC1" pad="3"/>
+<wire x1="37.084" y1="47.752" x2="40.005" y2="50.673" width="0.4064" layer="16"/>
+<wire x1="40.005" y1="50.673" x2="46.101" y2="50.673" width="0.4064" layer="16"/>
+<wire x1="46.101" y1="50.673" x2="46.609" y2="50.165" width="0.4064" layer="16"/>
+<wire x1="46.609" y1="50.165" x2="46.609" y2="47.752" width="0.4064" layer="16"/>
+<wire x1="46.609" y1="47.752" x2="45.847" y2="46.99" width="0.4064" layer="16"/>
+<wire x1="45.847" y1="46.99" x2="44.45" y2="46.99" width="0.4064" layer="16"/>
 </signal>
 <signal name="IACA_IN">
-<contactref element="IC1" pad="3"/>
 <contactref element="R1" pad="1"/>
 <contactref element="INPUT" pad="1"/>
-<wire x1="41.529" y1="45.974" x2="43.434" y2="45.974" width="0.4064" layer="16"/>
-<wire x1="43.434" y1="45.974" x2="44.45" y2="46.99" width="0.4064" layer="16"/>
 <wire x1="40.3606" y1="25.908" x2="40.3606" y2="30.1244" width="0.4064" layer="16"/>
 <wire x1="40.3606" y1="30.1244" x2="38.862" y2="31.623" width="0.4064" layer="16"/>
 <wire x1="38.862" y1="31.623" x2="38.862" y2="43.307" width="0.4064" layer="16"/>
 <wire x1="38.862" y1="43.307" x2="41.529" y2="45.974" width="0.4064" layer="16"/>
+<contactref element="IC1" pad="2"/>
+<wire x1="41.529" y1="45.974" x2="41.529" y2="48.641" width="0.4064" layer="16"/>
+<wire x1="41.529" y1="48.641" x2="42.418" y2="49.53" width="0.4064" layer="16"/>
+<wire x1="42.418" y1="49.53" x2="44.45" y2="49.53" width="0.4064" layer="16"/>
 </signal>
 <signal name="IACB_OUT">
@@
 </signal>
 <signal name="IACD_OUT">
-<contactref element="IC1" pad="15"/>
 <contactref element="OUTPUT" pad="4"/>
-<wire x1="52.07" y1="49.53" x2="55.245" y2="49.53" width="0.4064" layer="16"/>
-<wire x1="55.245" y1="49.53" x2="59.182" y2="45.593" width="0.4064" layer="16"/>
 <wire x1="59.182" y1="21.1836" x2="55.5244" y2="17.526" width="0.4064" layer="16"/>
-<wire x1="59.182" y1="45.593" x2="59.182" y2="21.1836" width="0.4064" layer="16"/>
+<wire x1="59.182" y1="47.244" x2="59.182" y2="21.1836" width="0.4064" layer="16"/>
+<contactref element="IC1" pad="14"/>
+<wire x1="59.182" y1="47.244" x2="55.753" y2="50.673" width="0.4064" layer="16"/>
+<wire x1="55.753" y1="50.673" x2="50.927" y2="50.673" width="0.4064" layer="16"/>
+<wire x1="50.927" y1="50.673" x2="50.038" y2="49.784" width="0.4064" layer="16"/>
+<wire x1="50.038" y1="49.784" x2="50.038" y2="47.371" width="0.4064" layer="16"/>
+<wire x1="50.038" y1="47.371" x2="50.419" y2="46.99" width="0.4064" layer="16"/>
+<wire x1="50.419" y1="46.99" x2="52.07" y2="46.99" width="0.4064" layer="16"/>
 </signal>
 <signal name="IACD_IN">
-<contactref element="IC1" pad="14"/>
 <contactref element="R4" pad="1"/>
 <contactref element="INPUT" pad="4"/>
@@
 <wire x1="55.3974" y1="29.6164" x2="57.912" y2="32.131" width="0.4064" layer="16"/>
 <wire x1="57.912" y1="42.926" x2="55.118" y2="45.72" width="0.4064" layer="16"/>
-<wire x1="52.07" y1="46.99" x2="53.848" y2="46.99" width="0.4064" layer="16"/>
-<wire x1="53.848" y1="46.99" x2="55.118" y2="45.72" width="0.4064" layer="16"/>
 <wire x1="57.912" y1="42.926" x2="57.912" y2="32.131" width="0.4064" layer="16"/>
+<contactref element="IC1" pad="15"/>
+<wire x1="55.118" y1="45.72" x2="55.118" y2="49.022" width="0.4064" layer="16"/>
+<wire x1="55.118" y1="49.022" x2="54.61" y2="49.53" width="0.4064" layer="16"/>
+<wire x1="54.61" y1="49.53" x2="52.07" y2="49.53" width="0.4064" layer="16"/>
 </signal>
 <signal name="IACC_OUT">
@@
 <signal name="N$1">
 <polygon width="0.4064" layer="16" isolate="0.6096">
-<vertex x="35.179" y="62.357"/>
-<vertex x="61.595" y="62.357"/>
+<vertex x="35.052" y="62.992"/>
+<vertex x="61.595" y="62.992"/>
 <vertex x="61.595" y="13.208"/>
 <vertex x="35.179" y="13.208"/>
