File: boards/PCB_Separated/platform_smd.brd (EAGLE design)
At the start: 100 x 80 mm, 94 parts, among them IC1 FT232RL, IC2 7805DT, IC4 L293D, IC5 7805DT, Q1 IRF3704S, Q2 IRF3704S, Q3 IRF3704S, Q4 IRF3704S, Q5 IRF3704S, U1 STM32F10XRXT6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

Commit message: run test again
Parts:
- R-ICU1, R-ICU6, R-VDDO: value 1k -> 330
Changed lines of the file:
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@@
 </element>
 <element name="TR-ICU" library="transistor" package="SOT23-BEC" value="" x="62.992" y="32.893" rot="MR0"/>
-<element name="R-ICU1" library="resistor" package="R0805" value="1k" x="63.119" y="26.162" rot="MR180"/>
+<element name="R-ICU1" library="resistor" package="R0805" value="330" x="63.119" y="26.162" rot="MR180"/>
 <element name="R-ICU2" library="resistor" package="R0805" value="4k7" x="63.119" y="28.067" rot="MR180"/>
 <element name="C-ICU" library="resistor" package="C0805" value="100n" x="63.119" y="29.972" rot="MR0"/>
@@
 <element name="C-VCC" library="resistor" package="PANASONIC_D" value="100u/25v" x="91.567" y="56.769" rot="MR0"/>
 <element name="TR-ICU1" library="transistor" package="SOT23-BEC" value="" x="58.42" y="33.02" rot="MR0"/>
-<element name="R-ICU6" library="resistor" package="R0805" value="1k" x="58.547" y="26.162" rot="MR180"/>
+<element name="R-ICU6" library="resistor" package="R0805" value="330" x="58.547" y="26.162" rot="MR180"/>
 <element name="R-ICU7" library="resistor" package="R0805" value="4k7" x="58.42" y="29.972" rot="MR180"/>
 <element name="C-ICU1" library="resistor" package="C0805" value="100n" x="58.42" y="28.067" rot="MR0"/>
 <element name="TR-VDDO" library="transistor" package="SOT23-BEC" value="" x="65.024" y="60.452" rot="MR0"/>
-<element name="R-VDDO" library="resistor" package="R0805" value="1k" x="67.691" y="58.039" rot="MR90"/>
+<element name="R-VDDO" library="resistor" package="R0805" value="330" x="67.691" y="58.039" rot="MR90"/>
 <element name="OKA1" library="optocoupler" package="DIL04" value="PC817" x="39.878" y="61.468" rot="R90">
 <attribute name="OC_NEWARK" value="97K7059" x="39.878" y="61.468" size="1.778" layer="27" rot="R90" display="off"/>
