File: boards/PCB_Separated/platform_smd.sch (EAGLE design)
At the start: 94 parts, among them IC1 FT232RL, IC2 7805DT, IC4 L293D, IC5 7805DT, Q1 IRF3704S, Q2 IRF3704S, Q3 IRF3704S, Q4 IRF3704S, Q5 IRF3704S, U1 STM32F10XRXT6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

Commit message: run test again
Parts:
- R-ICU1, R-ICU6, R-VDDO: value 1k -> 330
Changed lines of the file:
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@@
 <part name="OK-ICU" library="optocoupler" deviceset="H11L*M" device="" technology="1"/>
 <part name="TR-ICU" library="transistor" deviceset="*-NPN-" device="SOT23-BEC" technology="MMBT3904LT1"/>
-<part name="R-ICU1" library="resistor" deviceset="R-EU_" device="R0805" value="1k"/>
+<part name="R-ICU1" library="resistor" deviceset="R-EU_" device="R0805" value="330"/>
 <part name="R-ICU2" library="resistor" deviceset="R-EU_" device="R0805" value="4k7"/>
 <part name="C-ICU" library="resistor" deviceset="C-EU" device="C0805" value="100n"/>
@@
 <part name="C-VCC" library="resistor" deviceset="CPOL-EU" device="D" value="100u/25v"/>
 <part name="TR-ICU1" library="transistor" deviceset="*-NPN-" device="SOT23-BEC" technology="MMBT3904LT1"/>
-<part name="R-ICU6" library="resistor" deviceset="R-EU_" device="R0805" value="1k"/>
+<part name="R-ICU6" library="resistor" deviceset="R-EU_" device="R0805" value="330"/>
 <part name="R-ICU7" library="resistor" deviceset="R-EU_" device="R0805" value="4k7"/>
 <part name="C-ICU1" library="resistor" deviceset="C-EU" device="C0805" value="100n"/>
 <part name="TR-VDDO" library="transistor" deviceset="*-NPN-" device="SOT23-BEC" technology="MMBT3904LT1"/>
-<part name="R-VDDO" library="resistor" deviceset="R-EU_" device="R0805" value="1k"/>
+<part name="R-VDDO" library="resistor" deviceset="R-EU_" device="R0805" value="330"/>
 <part name="OKA1" library="optocoupler" deviceset="PC817" device=""/>
 <part name="OKA2" library="optocoupler" deviceset="PC817" device=""/>
