File: boards/PCB_Separated/platform_smd2_driver.brd (EAGLE design)
At the start: 100 x 80 mm, 14 parts

Commit message: fix some bugs
Parts:
- moved OUTPUT 0.64 mm to (18.4, 43.2), turned to 90 degrees
Connections:
- net IGNO1 renamed IGN1O
- net IGNO2 renamed INJ2O
- net INJO2 renamed IGN2O
- removed net INJO1: OUT.1, Q-INJ1.2, R-INJ1.1
- new net INJ1O: OUT.5, Q-PUMP.2, R-PUMP.1
- net IGN2: now also Q-INJ2.1; no longer Q-IGN2.1
- net INJ1: now also Q-PUMP.1; no longer Q-INJ1.1
- net INJ2: now also Q-IGN2.1; no longer Q-INJ2.1
- net PUMP: now also Q-INJ1.1; no longer Q-PUMP.1
- net PUMPO: now also OUT.1, Q-INJ1.2, R-INJ1.1; no longer OUT.5, Q-PUMP.2, R-PUMP.1
Routing:
- net INJO1: track 30.9 -> 0.00 mm
- net INJ1O: track 0.00 -> 25.1 mm
- net PUMPO: track 25.3 -> 30.9 mm
- net INJ1: track 27.1 -> 30.3 mm
- net PUMP: track 30.0 -> 26.9 mm
- net INJ2: track 16.4 -> 19.4 mm
- net IGN2: track 19.5 -> 17.1 mm
- net IGN1: track 11.6 -> 12.2 mm
