File: boards/PCB_Separated/platform_smd2_map2.brd (EAGLE design)
At the start: 100 x 80 mm, 62 parts, among them IC1 FT232RL, IC2 7805DT, U1 STM32F10XRXT6, X0 PN61729-S, X1 32khz, X2 8mhz

Commit message: perbaikan desain board
Parts:
- removed R-VDDO: 330, resistor:R0805
- removed X0: PN61729-S, con-berg:PN61729-S
- added C-VDDO: 100n, resistor:C1206
- added R-VDDO1, R-VDDO2: 4k7, resistor:M1206
- added X3: MINI-USB-32005-201, con-cypressindustries:32005-201
- L-ICU: device led:SML0805 -> led:1206
- moved TR-VDDO 41.4 mm to (41.3, 22.9)
- moved R-ICU1 1.27 mm to (54.0, 23.5)
- moved R-ICU2 0.63 mm to (54.0, 26.7)
- turned L-ICU to 270 degrees
- turned PWR-IN to 270 degrees
Connections:
- removed net N$19: R-VDDO.2, TR-VDDO.B
- net DM: now also X3.2; no longer X0.2
- net DP: now also X3.3; no longer X0.3
- net P35: now also C-VDDO.1, R-VDDO1.2, TR-VDDO.B
- net P58: no longer R-VDDO.1
- net VCC: now also X3.1; no longer X0.1
- net VDD: now also R-VDDO1.1, R-VDDO2.2; no longer TR-VDDO.C
- net VDDO: now also R-VDDO2.1, TR-VDDO.C; no longer TR-VDDO.E
- net VSS: now also C-VDDO.2, TR-VDDO.E, X3.5; no longer X0.4, X0.S1, X0.S2
Routing:
- net VDD: track 163.7 -> 268.4 mm, vias 4 -> 10
- net VSS: track 353.6 -> 451.8 mm, vias 8 -> 4
- net V12: track 171.3 -> 246.9 mm, vias 8 -> 0
- net GND: track 156.3 -> 210.6 mm, vias 0 -> 2
- net VDDO: track 130.9 -> 85.5 mm, vias 4 -> 0
- net VCC: track 122.6 -> 161.0 mm, vias 2 -> 4
- net P35: track 0.00 -> 32.3 mm
- net P58: track 12.4 -> 0.00 mm
- net INJ1: track 25.9 -> 16.1 mm
- net DM: track 4.80 -> 11.0 mm
- net IN: track 15.4 -> 20.9 mm
- net PUMP: track 23.8 -> 18.7 mm
- net P41: track 30.0 -> 26.8 mm
- net N$5: track 9.62 -> 12.7 mm
- net ICU: track 6.96 -> 10.0 mm
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
Commit message: coolant measurement
Parts:
- R-CLT1: value 1k -> 4k7
Changed lines of the file:
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@@
 <element name="R-MAT2" library="resistor" package="R1206" value="1k" x="74.295" y="25.4" rot="MR0"/>
 <element name="C-MAT" library="resistor" package="C1206" value="100n" x="74.295" y="22.86" rot="MR180"/>
-<element name="R-CLT1" library="resistor" package="R1206" value="1k" x="74.295" y="20.32" rot="MR0"/>
+<element name="R-CLT1" library="resistor" package="R1206" value="4k7" x="74.295" y="20.32" rot="MR0"/>
 <element name="R-CLT2" library="resistor" package="R1206" value="1k" x="74.295" y="17.78" rot="MR0"/>
 <element name="C-CLT" library="resistor" package="C1206" value="100n" x="74.295" y="15.24" rot="MR180"/>
