File: boards/PCB_Separated/platform_smd2_map2.sch (EAGLE design)
At the start: 64 parts, among them IC1 FT232RL, IC2 7805DT, U1 STM32F10XRXT6, X1 32khz, X2 8mhz, X3 MINI-USB-32005-201

Commit message: coolant measurement
Parts:
- R-CLT1: value 1k -> 4k7
Changed lines of the file:
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@@
 <part name="R-MAT2" library="resistor" deviceset="R-EU_" device="R1206" value="1k"/>
 <part name="C-MAT" library="resistor" deviceset="C-EU" device="C1206" value="100n"/>
-<part name="R-CLT1" library="resistor" deviceset="R-EU_" device="R1206" value="1k"/>
+<part name="R-CLT1" library="resistor" deviceset="R-EU_" device="R1206" value="4k7"/>
 <part name="R-CLT2" library="resistor" deviceset="R-EU_" device="R1206" value="1k"/>
 <part name="C-CLT" library="resistor" deviceset="C-EU" device="C1206" value="100n"/>
