File: boards/PCB_Separated/platform_all1.sch (EAGLE design)
At the start: 80 parts, among them IC1 FT232RL, IC2 7805DT, IC3 7805DT, U1 STM32F10XRXT6, X1 32khz, X2 8mhz, X3 MINI-USB_SHIELD5P2-32005-601

Commit message: edit mini usb and deactivate delayed startup
Parts:
- removed X3: MINI-USB_SHIELD5P2-32005-601, con-cypressindustries:MINI-USB_SHIELD5P2-32005-601
- added USB: MINI-USB-32005-201, con-cypressindustries:MINI-USB-32005-201
Connections:
- net DM: now also USB.2; no longer X3G41.2
- net DP: now also USB.3; no longer X3G41.3
- net VCC: now also USB.1; no longer X3G41.1
- net VSS: now also USB.5; no longer X3G41.5
Changed lines of the file:
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@@
 <part name="R-CLT2" library="resistor" deviceset="R-EU_" device="R1206" value="1k"/>
 <part name="C-CLT" library="resistor" deviceset="C-EU" device="C1206" value="100n"/>
-<part name="X3" library="con-cypressindustries" deviceset="MINI-USB_SHIELD5P2-" device="32005-601"/>
 <part name="R-O21" library="resistor" deviceset="R-EU_" device="R1206" value="1k"/>
 <part name="R-O22" library="resistor" deviceset="R-EU_" device="R1206" value="1k"/>
@@
 <part name="CON1" library="pinhead" deviceset="PINHD-1X12" device=""/>
 <part name="CON2" library="pinhead" deviceset="PINHD-1X12" device=""/>
+<part name="USB" library="con-cypressindustries" deviceset="MINI-USB-" device="32005-201"/>
 </parts>
 <sheets>
@@
 <instance part="R-CLT2" gate="G$1" x="10.16" y="-121.92" rot="R90"/>
 <instance part="C-CLT" gate="G$1" x="15.24" y="-119.38"/>
-<instance part="X3" gate="G41" x="162.56" y="48.26"/>
 <instance part="R-O21" gate="G$1" x="-48.26" y="-137.16"/>
 <instance part="R-O22" gate="G$1" x="-40.64" y="-144.78" rot="R90"/>
@@
 <instance part="CON1" gate="G$1" x="233.68" y="-17.78" rot="R180"/>
 <instance part="CON2" gate="G$1" x="238.76" y="-58.42"/>
+<instance part="USB" gate="G$1" x="162.56" y="25.4"/>
 </instances>
 <busses>
@@
 </segment>
 <segment>
-<pinref part="X3" gate="G41" pin="5"/>
-<wire x1="157.48" y1="43.18" x2="149.86" y2="43.18" width="0.1524" layer="91"/>
-<label x="144.78" y="43.18" size="1.778" layer="95"/>
-</segment>
-<segment>
 <pinref part="C-O2" gate="G$1" pin="2"/>
 <wire x1="-35.56" y1="-147.32" x2="-35.56" y2="-152.4" width="0.1524" layer="91"/>
@@
 <wire x1="10.16" y1="-152.4" x2="10.16" y2="-149.86" width="0.1524" layer="91"/>
 <label x="15.24" y="-152.4" size="1.778" layer="95"/>
+</segment>
+<segment>
+<pinref part="USB" gate="G$1" pin="5"/>
+<wire x1="157.48" y1="20.32" x2="149.86" y2="20.32" width="0.1524" layer="91"/>
+<label x="144.78" y="20.32" size="1.778" layer="95"/>
 </segment>
 </net>
@@
 </segment>
 <segment>
-<pinref part="X3" gate="G41" pin="1"/>
-<wire x1="157.48" y1="53.34" x2="149.86" y2="53.34" width="0.1524" layer="91"/>
-<label x="144.78" y="53.34" size="1.778" layer="95"/>
-</segment>
-<segment>
 <pinref part="ANALOG" gate="-1" pin="KL"/>
 <wire x1="-96.52" y1="-68.58" x2="-88.9" y2="-68.58" width="0.1524" layer="91"/>
 <label x="-91.44" y="-68.58" size="1.778" layer="95"/>
 </segment>
+<segment>
+<pinref part="USB" gate="G$1" pin="1"/>
+<wire x1="157.48" y1="30.48" x2="149.86" y2="30.48" width="0.1524" layer="91"/>
+<label x="144.78" y="30.48" size="1.778" layer="95"/>
+</segment>
 </net>
 <net name="DP" class="0">
@@
 </segment>
 <segment>
-<pinref part="X3" gate="G41" pin="3"/>
-<wire x1="157.48" y1="48.26" x2="149.86" y2="48.26" width="0.1524" layer="91"/>
-<label x="144.78" y="48.26" size="1.778" layer="95"/>
+<pinref part="USB" gate="G$1" pin="3"/>
+<wire x1="157.48" y1="25.4" x2="149.86" y2="25.4" width="0.1524" layer="91"/>
+<label x="144.78" y="25.4" size="1.778" layer="95"/>
 </segment>
 </net>
@@
 </segment>
 <segment>
-<pinref part="X3" gate="G41" pin="2"/>
-<wire x1="157.48" y1="50.8" x2="149.86" y2="50.8" width="0.1524" layer="91"/>
-<label x="144.78" y="50.8" size="1.778" layer="95"/>
-</segment>
-</net>
+<pinref part="USB" gate="G$1" pin="2"/>
+<wire x1="157.48" y1="27.94" x2="149.86" y2="27.94" width="0.1524" layer="91"/>
+<label x="144.78" y="27.94" size="1.778" layer="95"/>
+</segment>
+</net>
